Commit message: Im done with pure mpc demos

File: legged_locomotion_mpc_ros2/include/legged_locomotion_mpc_ros2/demos/meldog_demo/meldog.urdf (robot description, URDF)
Before this commit: robot meldog_core, 18 links, 17 joints
Links:
- link LFLL_link: geometry collision cylinder length=0.25 radius=0.0275
- link LRLL_link: geometry collision cylinder length=0.25 radius=0.0275
- link RFLL_link: geometry collision cylinder length=0.25 radius=0.0275
- link RRLL_link: geometry collision cylinder length=0.25 radius=0.0275

Commit message: Added collision links, demos fixed

File: legged_locomotion_mpc_ros2/include/legged_locomotion_mpc_ros2/demos/meldog_demo/meldog.urdf (robot description, URDF)
Before this commit: robot meldog_core, 18 links, 17 joints
Links:
- link LFLL_link: geometry collision cylinder length=0.15 radius=0.0275
- link LRLL_link: geometry collision cylinder length=0.15 radius=0.0275
- link RFLL_link: geometry collision cylinder length=0.15 radius=0.0275
- link RRLL_link: geometry collision cylinder length=0.15 radius=0.0275
